File: cosmic_ray_detector/frontend.kicad_sch (KiCad schematic)
At the start: 15 parts, among them U1 TL072

Commit message: many more footprints coming in
Parts:
- C2: value C_Polarized_US -> (none); Farnell (none) -> 1187014; MPN (none) -> MAL215375109E3; Manufacturer_Name (none) -> Vishay
- C3: value ~ -> (none); Farnell (none) -> 1187014; MPN (none) -> MAL215375109E3; Manufacturer_Name (none) -> Vishay
- C4, C6: value C -> (none)
- C5, C7, C8, R3, R4: value ~ -> (none)
- D1: value VBPW34FAS -> (none)
- R2: value R_US -> (none)
- TP1: value TestPoint -> (none); Farnell (none) -> 2293786; MPN (none) -> S1751-46R; Manufacturer_Name (none) -> Harwin
- TP2, TP3: value ~ -> (none); Farnell (none) -> 2293786; MPN (none) -> S1751-46R; Manufacturer_Name (none) -> Harwin
- U1: value TL072 -> (none); Farnell (none) -> 1467663; MPN (none) -> TL072CDT
Changed lines of the file:
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@@
     (in_bom yes) (on_board yes) (fields_autoplaced)
     (property "Reference" "U1" (id 0) (at 219.71 97.79 0))
-    (property "Value" "TL072" (id 1) (at 219.71 100.33 0))
+    (property "Value" "" (id 1) (at 219.71 100.33 0))
     (property "Footprint" "" (id 2) (at 219.71 107.95 0)
       (effects (font (size 1.27 1.27)) hide)
     )
     (property "Datasheet" "http://www.ti.com/lit/ds/symlink/tl071.pdf" (id 3) (at 219.71 107.95 0)
+      (effects (font (size 1.27 1.27)) hide)
+    )
+    (property "MPN" "TL072CDT" (id 4) (at 219.71 107.95 0)
+      (effects (font (size 1.27 1.27)) hide)
+    )
+    (property "farnell" "" (id 5) (at 219.71 107.95 0)
+      (effects (font (size 1.27 1.27)) hide)
+    )
+    (property "Farnell" "1467663 " (id 6) (at 219.71 107.95 0)
       (effects (font (size 1.27 1.27)) hide)
     )
@@
     (in_bom yes) (on_board yes)
     (property "Reference" "R4" (id 0) (at 220.98 78.74 90))
-    (property "Value" "~" (id 1) (at 217.17 76.2 90))
+    (property "Value" "" (id 1) (at 217.17 76.2 90))
     (property "Footprint" "" (id 2) (at 217.424 78.994 90)
       (effects (font (size 1.27 1.27)) hide)
@@
     (in_bom yes) (on_board yes) (fields_autoplaced)
     (property "Reference" "C7" (id 0) (at 194.31 97.79 90))
-    (property "Value" "~" (id 1) (at 194.31 100.33 90))
+    (property "Value" "" (id 1) (at 194.31 100.33 90))
     (property "Footprint" "" (id 2) (at 198.12 104.4448 0)
       (effects (font (size 1.27 1.27)) hide)
@@
     (in_bom yes) (on_board yes) (fields_autoplaced)
     (property "Reference" "R2" (id 0) (at 129.54 72.39 90))
-    (property "Value" "R_US" (id 1) (at 129.54 74.93 90))
+    (property "Value" "" (id 1) (at 129.54 74.93 90))
     (property "Footprint" "" (id 2) (at 129.794 77.724 90)
       (effects (font (size 1.27 1.27)) hide)
@@
       (effects (font (size 1.27 1.27)) (justify left))
     )
-    (property "Value" "VBPW34FAS" (id 1) (at 57.15 82.5499 90)
+    (property "Value" "" (id 1) (at 57.15 82.5499 90)
       (effects (font (size 1.27 1.27)) (justify left))
     )
@@
       (effects (font (size 1.27 1.27)) (justify left))
     )
-    (property "Value" "C" (id 1) (at 60.96 163.8299 0)
+    (property "Value" "" (id 1) (at 60.96 163.8299 0)
       (effects (font (size 1.27 1.27)) (justify left))
     )
@@
       (effects (font (size 1.27 1.27)) (justify left))
     )
-    (property "Value" "~" (id 1) (at 50.8 175.8949 0)
+    (property "Value" "" (id 1) (at 50.8 175.8949 0)
       (effects (font (size 1.27 1.27)) (justify left))
     )
@@
       (effects (font (size 1.27 1.27)) hide)
     )
+    (property "Farnell" "1187014 " (id 4) (at 46.99 175.26 0)
+      (effects (font (size 1.27 1.27)) hide)
+    )
+    (property "MPN" "MAL215375109E3" (id 5) (at 46.99 175.26 0)
+      (effects (font (size 1.27 1.27)) hide)
+    )
+    (property "Manufacturer_Name" "Vishay" (id 6) (at 46.99 175.26 0)
+      (effects (font (size 1.27 1.27)) hide)
+    )
     (pin "1")
     (pin "2")
@@
     (in_bom yes) (on_board yes) (fields_autoplaced)
     (property "Reference" "R3" (id 0) (at 184.15 99.06 90))
-    (property "Value" "~" (id 1) (at 184.15 101.6 90))
+    (property "Value" "" (id 1) (at 184.15 101.6 90))
     (property "Footprint" "" (id 2) (at 184.404 104.394 90)
       (effects (font (size 1.27 1.27)) hide)
@@
     (in_bom yes) (on_board yes)
     (property "Reference" "C8" (id 0) (at 219.71 88.9 90))
-    (property "Value" "~" (id 1) (at 217.17 85.09 90))
+    (property "Value" "" (id 1) (at 217.17 85.09 90))
     (property "Footprint" "" (id 2) (at 220.98 89.2048 0)
       (effects (font (size 1.27 1.27)) hide)
@@
       (effects (font (size 1.27 1.27)) (justify left))
     )
-    (property "Value" "C_Polarized_US" (id 1) (at 46.99 163.1949 0)
+    (property "Value" "" (id 1) (at 46.99 163.1949 0)
       (effects (font (size 1.27 1.27)) (justify left))
     )
@@
       (effects (font (size 1.27 1.27)) hide)
     )
+    (property "Farnell" "1187014 " (id 4) (at 43.18 162.56 0)
+      (effects (font (size 1.27 1.27)) hide)
+    )
+    (property "MPN" "MAL215375109E3" (id 5) (at 43.18 162.56 0)
+      (effects (font (size 1.27 1.27)) hide)
+    )
+    (property "Manufacturer_Name" "Vishay" (id 6) (at 43.18 162.56 0)
+      (effects (font (size 1.27 1.27)) hide)
+    )
     (pin "1")
     (pin "2")
@@
     (in_bom yes) (on_board yes) (fields_autoplaced)
     (property "Reference" "C6" (id 0) (at 129.54 57.15 90))
-    (property "Value" "C" (id 1) (at 129.54 59.69 90))
+    (property "Value" "" (id 1) (at 129.54 59.69 90))
     (property "Footprint" "" (id 2) (at 133.35 63.8048 0)
       (effects (font (size 1.27 1.27)) hide)
@@
       (effects (font (size 1.27 1.27)) (justify left))
     )
-    (property "Value" "TestPoint" (id 1) (at 99.06 100.8379 0)
+    (property "Value" "" (id 1) (at 99.06 100.8379 0)
       (effects (font (size 1.27 1.27)) (justify left))
     )
@@
     )
     (property "Datasheet" "~" (id 3) (at 102.235 102.87 0)
+      (effects (font (size 1.27 1.27)) hide)
+    )
+    (property "Farnell" "2293786" (id 4) (at 97.155 102.87 0)
+      (effects (font (size 1.27 1.27)) hide)
+    )
+    (property "MPN" "S1751-46R" (id 5) (at 97.155 102.87 0)
+      (effects (font (size 1.27 1.27)) hide)
+    )
+    (property "Manufacturer_Name" "Harwin" (id 6) (at 97.155 102.87 0)
       (effects (font (size 1.27 1.27)) hide)
     )
@@
       (effects (font (size 1.27 1.27)) (justify left))
     )
-    (property "Value" "~" (id 1) (at 60.96 176.5299 0)
+    (property "Value" "" (id 1) (at 60.96 176.5299 0)
       (effects (font (size 1.27 1.27)) (justify left))
     )
@@
       (effects (font (size 1.27 1.27)) (justify left))
     )
-    (property "Value" "~" (id 1) (at 169.037 103.3779 0)
+    (property "Value" "" (id 1) (at 169.037 103.3779 0)
       (effects (font (size 1.27 1.27)) (justify left))
     )
@@
       (effects (font (size 1.27 1.27)) hide)
     )
+    (property "Farnell" "2293786" (id 4) (at 167.132 105.41 0)
+      (effects (font (size 1.27 1.27)) hide)
+    )
+    (property "MPN" "S1751-46R" (id 5) (at 167.132 105.41 0)
+      (effects (font (size 1.27 1.27)) hide)
+    )
+    (property "Manufacturer_Name" "Harwin" (id 6) (at 167.132 105.41 0)
+      (effects (font (size 1.27 1.27)) hide)
+    )
     (pin "1")
   )
@@
     (in_bom yes) (on_board yes) (fields_autoplaced)
     (property "Reference" "U1" (id 0) (at 125.73 95.25 0))
-    (property "Value" "TL072" (id 1) (at 125.73 97.79 0))
+    (property "Value" "" (id 1) (at 125.73 97.79 0))
     (property "Footprint" "" (id 2) (at 125.73 105.41 0)
       (effects (font (size 1.27 1.27)) hide)
     )
     (property "Datasheet" "http://www.ti.com/lit/ds/symlink/tl071.pdf" (id 3) (at 125.73 105.41 0)
+      (effects (font (size 1.27 1.27)) hide)
+    )
+    (property "MPN" "TL072CDT" (id 4) (at 125.73 105.41 0)
+      (effects (font (size 1.27 1.27)) hide)
+    )
+    (property "farnell" "" (id 5) (at 125.73 105.41 0)
+      (effects (font (size 1.27 1.27)) hide)
+    )
+    (property "Farnell" "1467663 " (id 6) (at 125.73 105.41 0)
       (effects (font (size 1.27 1.27)) hide)
     )
@@
       (effects (font (size 1.27 1.27)) (justify left))
     )
-    (property "Value" "TL072" (id 1) (at 77.47 170.1799 0)
+    (property "Value" "" (id 1) (at 77.47 170.1799 0)
       (effects (font (size 1.27 1.27)) (justify left))
     )
@@
     )
     (property "Datasheet" "http://www.ti.com/lit/ds/symlink/tl071.pdf" (id 3) (at 78.74 168.91 0)
+      (effects (font (size 1.27 1.27)) hide)
+    )
+    (property "MPN" "TL072CDT" (id 4) (at 78.74 168.91 0)
+      (effects (font (size 1.27 1.27)) hide)
+    )
+    (property "farnell" "" (id 5) (at 78.74 168.91 0)
+      (effects (font (size 1.27 1.27)) hide)
+    )
+    (property "Farnell" "1467663 " (id 6) (at 78.74 168.91 0)
       (effects (font (size 1.27 1.27)) hide)
     )
@@
       (effects (font (size 1.27 1.27)) (justify left))
     )
-    (property "Value" "~" (id 1) (at 240.665 105.9179 0)
+    (property "Value" "" (id 1) (at 240.665 105.9179 0)
       (effects (font (size 1.27 1.27)) (justify left))
     )
@@
       (effects (font (size 1.27 1.27)) hide)
     )
+    (property "Farnell" "2293786" (id 4) (at 238.76 107.95 0)
+      (effects (font (size 1.27 1.27)) hide)
+    )
+    (property "MPN" "S1751-46R" (id 5) (at 238.76 107.95 0)
+      (effects (font (size 1.27 1.27)) hide)
+    )
+    (property "Manufacturer_Name" "Harwin" (id 6) (at 238.76 107.95 0)
+      (effects (font (size 1.27 1.27)) hide)
+    )
