File: frontend_sim/frontend_sim.kicad_sch (KiCad schematic)
At the start: 12 parts

Commit message: sim work
Parts:
- removed C3, C4: (no value), symbol pspice:C
- added C3, C4: (no value), symbol pspice:CAP
- added R4: (no value), symbol pspice:R
- added U3: (no value), symbol pspice:OPAMP
- added V3: (no value), symbol pspice:VSOURCE
- C2: Spice_Model (none) -> 2p; Spice_Netlist_Enabled (none) -> Y; Spice_Primitive (none) -> C
- I1: Spice_Model ac 10p -> dc 0 ac 10n pulse(0 -100p 1n 100p 100p 1u)
- R1: Spice_Model 1Meg -> 100Meg
- R2: Spice_Model R -> 100; Spice_Netlist_Enabled N -> Y
- R3: Spice_Model R -> 100Meg; Spice_Netlist_Enabled N -> Y
- U1: value (none) -> TL072
- U2: Spice_Lib_File (none) -> TL072.301; Spice_Model (none) -> TL072; Spice_Netlist_Enabled N -> Y; Spice_Node_Sequence (none) -> 1 2 4 5 3; Spice_Primitive R -> X
- V1, V2: value (none) -> VSOURCE
Connections:
- net +5VA: now also U2.4 (V+), U3.4 (V+)
- net -5VA: now also U2.5 (V-), U3.5 (V-)
- net 0: now also U2.1 (+), R4.1, V3.2 (E2); no longer U2.2 (-)
- net CSA_FB: now also C3.1
- net at R2.1: now also C3.2
- net at R2.2, R3.1: now also U2.2 (-), C4.1; no longer U2.1 (+)
- net CRRC_FB: now reaches R3.2, U2.3
- net CRRC_FB: now also C4.2, U3.1 (+)
- new net: U3.2 (-), V3.1 (E1)
- new net COMP_OUT: R4.2, U3.3

Commit message: updates to the simulation workbook for v9
Parts:
- C1: value (none) -> 10pF
- C2: value (none) -> 1pF; Spice_Model 2p -> (none); Spice_Netlist_Enabled Y -> (none); Spice_Primitive C -> (none)
- C3: value (none) -> 10n; Spice_Model 10n -> (none); Spice_Netlist_Enabled Y -> (none); Spice_Primitive C -> (none)
- C4: value (none) -> 100p; Spice_Model 10p -> (none); Spice_Netlist_Enabled Y -> (none); Spice_Primitive C -> (none)
- I1: value (none) -> ISOURCE; Spice_Model dc 0 ac 10n pulse(0 -100p 1n 100p 100p 1u) -> (none); Spice_Netlist_Enabled Y -> (none); Spice_Primitive I -> (none)
- R1: value (none) -> 100Meg; Spice_Model 100Meg -> (none); Spice_Netlist_Enabled Y -> (none); Spice_Primitive R -> (none)
- R2: value (none) -> 100; Spice_Model 100 -> (none); Spice_Netlist_Enabled Y -> (none); Spice_Primitive R -> (none)
- R3: value (none) -> 10Meg; Spice_Model 100Meg -> (none); Spice_Netlist_Enabled Y -> (none); Spice_Primitive R -> (none)
- R4: value (none) -> 50; Spice_Model 50 -> (none); Spice_Netlist_Enabled Y -> (none); Spice_Primitive R -> (none)
- U1: Spice_Lib_File TL072.301 -> (none); Spice_Model TL072 -> (none); Spice_Netlist_Enabled Y -> (none); Spice_Node_Sequence 1 2 4 5 3 -> (none); Spice_Primitive X -> (none)
- U2: value (none) -> TL072; Spice_Lib_File TL072.301 -> (none); Spice_Model TL072 -> (none); Spice_Netlist_Enabled Y -> (none); Spice_Node_Sequence 1 2 4 5 3 -> (none); Spice_Primitive X -> (none)
- U3: value (none) -> TLV3501; Spice_Lib_File tlv3501.lib -> (none); Spice_Model TLV3501 -> (none); Spice_Netlist_Enabled Y -> (none); Spice_Node_Sequence 1 2 4 4 5 3 -> (none); Spice_Primitive X -> (none)
- V1: value VSOURCE -> 5; Spice_Model dc 5 -> (none); Spice_Netlist_Enabled Y -> (none); Spice_Primitive V -> (none)
- V2: value VSOURCE -> -5; Spice_Model dc -5 -> (none); Spice_Netlist_Enabled Y -> (none); Spice_Primitive V -> (none)
- V3: value (none) -> 20m; Spice_Model dc 10m -> (none); Spice_Netlist_Enabled Y -> (none); Spice_Primitive V -> (none)
